File: DarkQuest_A5202_Crate_Backplate/rev1.1/cmos_switched_attenuator.kicad_sch (KiCad schematic)
At the start: 9 parts, among them U1 TMUX7612RUMR

Commit message: Fix net class widths, refdes numbering
Parts:
- renumbered C2 to C2A2, C3 to C2B2, R3A1 to R3A2, R3B1 to R3B2, R3C1 to R3C2, R3D1 to R3D2, R4A1 to R4A2, R4B1 to R4B2, U1 to U2
